Commit message: Implement LeRobot SmolVLA URDF pipeline with 1-DOF gripper, PyBullet env, tests, and eval videos

File: urdf/robot.urdf (robot description, URDF)
Before this commit: robot robot_4dof, 5 links, 4 joints
Links:
- added link gripper_base, mass 0.12; collision box size=0.06 0.08 0.02; visual box size=0.06 0.08 0.02
- added link gripper_left, mass 0.04; collision box size=0.012 0.012 0.06; visual box size=0.012 0.012 0.06
- added link gripper_right, mass 0.04; collision box size=0.012 0.012 0.06; visual box size=0.012 0.012 0.06
- link base_link: mass 1.0 -> 2.0; geometry collision cylinder length=0.05 radius=0.08; visual cylinder length=0.05 radius=0.08
- link ee_link: mass 0.1 -> 0.08; geometry collision sphere radius=0.018; visual sphere radius=0.02
- link link1: mass 0.5 -> 0.6; geometry collision cylinder length=0.2 radius=0.03; visual cylinder length=0.2 radius=0.03
- link link2: geometry collision box size=0.05 0.05 0.2; visual box size=0.05 0.05 0.2
- link link3: mass 0.5 -> 0.4; geometry collision box size=0.045 0.045 0.2; visual box size=0.045 0.045 0.2
Joints:
- added joint gripper_base_joint: type fixed, parent ee_link, child gripper_base, origin xyz=0 0 0.03
- added joint gripper_left_joint: type prismatic, parent gripper_base, child gripper_left, origin xyz=0.02 -0.038 0.03, axis 0 1 0, limit lower=0 upper=0.022 effort=30 velocity=0.2
- added joint gripper_right_joint: type prismatic, parent gripper_base, child gripper_right, origin xyz=0.02 0.038 0.03, axis 0 -1 0, limit lower=0 upper=0.022 effort=30 velocity=0.2
- joint joint1: limit lower=-3.14 upper=3.14 effort=10 velocity=1 -> lower=-3.1416 upper=3.1416 effort=20 velocity=2
- joint joint2: limit lower=-1.57 upper=1.57 effort=10 velocity=1 -> lower=-1.57 upper=1.57 effort=20 velocity=2
- joint joint3: limit lower=-1.57 upper=1.57 effort=10 velocity=1 -> lower=-1.57 upper=1.57 effort=20 velocity=2
- joint joint4: limit lower=-3.14 upper=3.14 effort=10 velocity=1 -> lower=-3.1416 upper=3.1416 effort=10 velocity=3
